Commit message: Minireto 2

File: ros2_ws/install/puzzlebot_sim/share/puzzlebot_sim/urdf/puzzlebot.urdf (robot description, URDF)
Before this commit: robot Puzzlebot_Jetson_Lidar_Ed., 0 links, 0 joints
Links:
- added link base_footprint
- added link base_link; visual mesh filename=package://puzzlebot_sim/meshes/MCR2_puzzlebot_jetson_lidar_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
- added link camera_base_link
- added link caster_holder_link; visual mesh filename=package://puzzlebot_sim/meshes/MCR2_caster_wheel.stl
- added link lidar_base_link
- added link wheel_left_link; visual mesh filename=package://puzzlebot_sim/meshes/MCR2_wheel.stl
- added link wheel_right_link; visual mesh filename=package://puzzlebot_sim/meshes/MCR2_wheel.stl
Joints:
- added joint base_link_joint: type fixed, parent base_footprint, child base_link, origin xyz=0 0 0.05 rpy=0 0 0
- added joint camera_base_joint: type fixed, parent base_link, child camera_base_link, origin xyz=0.112 0 0.065 rpy=0 0 0
- added joint caster_holder_joint: type fixed, parent base_link, child caster_holder_link, origin xyz=-0.095 0 -0.0307 rpy=0 0 0
- added joint lidar_base_joint: type fixed, parent base_link, child lidar_base_link, origin xyz=0.05 0 0.110 rpy=0 0 0
- added joint wheel_left_joint: type continuous, parent base_link, child wheel_left_link, origin xyz=0.052 0.095 -0.0025 rpy=0 0 0, axis 0 1 0
- added joint wheel_right_joint: type continuous, parent base_link, child wheel_right_link, origin xyz=0.052 -0.095 -0.0025 rpy=0 0 0, axis 0 1 0
